File: maiconvert-io4-breakout-board.kicad_pcb (KiCad board)
At the start: 2 copper layers, 170.8 x 114.6 mm, 96 parts, among them J1 CN3 - From IO4, J10 1P B7, J11 1P B8, J12 2P B1, J13 2P B2, J14 2P B3, J15 2P B4, J16 2P B5, J17 2P B6, J18 2P B7, J19 2P B8, J2 CN9 - From IO4, J20 1P SELECT BUTTON, J21 2P SELECT BUTTON, J22 12V input, J23 BILLBOARD LED L, J24 BILLBOARD LED R, J25 1P CODE READER LED, J26 2P CODE READER LED, J27 COIN METER, J28 COIN LOCKOUT, J29 CAMERA LED RED, J3 CN3 - To Harness (Passthrough), J30 CAMERA LED WARM, J31 TEST BUTTON, J32 COIN BUTTON, J33 SERVICE BUTTON, J34 EXV-5V Jumper, J35 Pin 51 Jumper, J4 1P B1, J5 1P B2, J6 1P B3, J7 1P B4, J8 1P B5, J9 1P B6, Q1 DMP3010LK3-13, SW1 TEST, SW10 1P B5 BTN, SW11 1P B6 BTN, SW12 1P B7 BTN, SW13 1P B8 BTN, SW14 2P B1 BTN, SW15 2P B2 BTN, SW16 2P B3 BTN, SW17 2P B4 BTN, SW18 2P B5 BTN, SW19 2P B6 BTN, SW2 COIN, SW20 2P B7 BTN, SW21 2P B8 BTN, SW3 SERVICE, SW4 1P SELECT BTN, SW5 2P SELECT BTN, SW6 1P B1 BTN, SW7 1P B2 BTN, SW8 1P B3 BTN, SW9 1P B4 BTN

Commit message: Final touches
Other:
- board text added: "For 1P 1-8, if no button is connected, put a jumper on pin 2 and 3, or tactile switches will not work"
- board text added: "For 2P 1-8, if no button is connected, put a jumper on pin 2 and 3, or tactile switches will not work"
- board text removed: "For 1P 1-8, if no button is connected, put a jumper on pin 2 and 3, or tactile switches will no work"
- board text removed: "For 2P 1-8, if no button is connected, put a jumper on pin 2 and 3, or tactile switches will no work"
Changed lines of the file:
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@@
 		)
 	)
-	(gr_text "For 1P 1-8, if no button is\nconnected, put a jumper on\npin 2 and 3, or tactile\nswitches will no work"
+	(gr_text "For 1P 1-8, if no button is\nconnected, put a jumper on\npin 2 and 3, or tactile\nswitches will not work"
 		(at 218.52 97.95 0)
 		(layer "F.SilkS")
@@
 		)
 	)
-	(gr_text "For 2P 1-8, if no button is\nconnected, put a jumper on\npin 2 and 3, or tactile\nswitches will no work"
+	(gr_text "For 2P 1-8, if no button is\nconnected, put a jumper on\npin 2 and 3, or tactile\nswitches will not work"
 		(at 218.61 70.88 0)
 		(layer "F.SilkS")
